File: PCB/Rev2.kicad_pcb (KiCad board)
At the start: 4 copper layers, 152.4 x 63.5 mm, 84 parts, among them J1 AudioJack, J2 Conn_01x03_Socket, J3 Conn_01x02_Pin, U1 TL974, U2 LM78M05, U3 SN76489, U4 TL974, U5 MCP42010, U6 SN76489

Commit message: Add files via upload
Changed default output voltage on receiver circuit. Added ground points, J4.
Parts:
- added J4: Conn_01x02_Pin, STFootPrints:PinHeader_1x02_P2.54mm_Vertical, F.Cu at (170.9, 65.8)
- R1, R13, R7: value 15K -> 56K
- R10, R16, R4: value 5M1 -> 1M8
- R11, R17, R5: value 100K -> 10K
- R14, R2, R8: value 15K -> 10K
- R15, R3, R9: value 100K -> 56K
- R22, R26, R30, R34: value 430K -> 300K
- U1: value TL974 -> LM324AN
Connections:
- net 12V renamed 16V
Other:
- board text added: "Rev 2.2"
- board text added: "Sterio Theremin Christle Engineering 2026"
- board text removed: "Rev 2.0"
- board text removed: "Ultra Sonic Theremin Christle Engineering 2026"
